File: PCB/CHIP_PRO-Dev-Kit-v1.0.sch (EAGLE design)
At the start: 121 parts, among them CN1 SJ-43514-SMT-TR, CN2 POWER_JACKPTH, J1 USB-MICROB, J2 USB_, Q1 MMBT2222A, Q10 MMBT2222A, Q2 MMBT2222A, Q3 MMBT2222A, Q4 MMBT2222A, Q5 MMBT2222A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

Commit message: update EAGLE library and source to fix errata in github issue #1
Connections:
- net TWI1-SCK: now also CHIP_PRO.TWI1-SDA, J3.11; no longer CHIP_PRO.TWI1-SCK, J3.12
- net TWI1-SDA: now also CHIP_PRO.TWI1-SCK, J3.12; no longer CHIP_PRO.TWI1-SDA, J3.11
Changed lines of the file:
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@@
 <?xml version="1.0" encoding="utf-8"?>
 <!DOCTYPE eagle SYSTEM "eagle.dtd">
-<eagle version="7.6.0">
+<eagle version="8.2.2">
 <drawing>
 <settings>
@@
 <setting verticaltext="up"/>
 </settings>
-<grid distance="50" unitdist="mil" unit="mil" style="lines" multiple="1" display="yes" altdistance="0.01" altunitdist="inch" altunit="inch"/>
+<grid distance="0.1" unitdist="inch" unit="inch" style="lines" multiple="1" display="no" altdistance="0.01" altunitdist="inch" altunit="inch"/>
 <layers>
 <layer number="1" name="Top" color="56" fill="1" visible="no" active="no"/>
@@
 </segment>
 </net>
-<net name="TWI1-SCK" class="0">
+<net name="TWI1-SDA" class="0">
 <segment>
 <pinref part="J3" gate="G$1" pin="12"/>
@@
 </segment>
 </net>
-<net name="TWI1-SDA" class="0">
+<net name="TWI1-SCK" class="0">
 <segment>
 <pinref part="J3" gate="G$1" pin="11"/>
